File: final/main_board.sch (KiCad schematic (older format))
At the start: 72 parts, among them J1 USB_microB_2040002-1, J2 Arduino_ICSP, J3 Conn_01x15_Male, J4 Conn_01x15_Male, J5 E-INK DISPLAY, J6 BT CONFIG, U1 FT232RL, U2 MCP1702T-5002E_CB, U3 TPS2113ADRBR, U4 ATMEGA328PB-ANR, U5 TXS0108EPW, U6 TXS0104E, U7 RN4871, U8 MCP1702T-3302E/CBCT-ND, U9 TS02CQE, Y1 16MHz

Commit message: Made Boards Better
Parts:
- removed C? (x2): 1µF, Capacitor_SMD:C_0603_1608Metric, symbol Device:C
- removed C?: 10µF, Capacitor_SMD:C_0603_1608Metric, symbol Device:C
- removed D3: PWR, LED_SMD:LED_0805_2012Metric, symbol Device:LED_ALT
- removed D?: LED, LED_SMD:LED_0805_2012Metric, symbol Device:LED_ALT
- removed J3, J4: Conn_01x15_Male, Connector_PinHeader_2.54mm:PinHeader_1x15_P2.54mm_Vertical, symbol Connector:Conn_01x15_Male
- removed R2: 10K, Resistor_SMD:R_0603_1608Metric, symbol Device:R
- removed R3, R?: 1K, Resistor_SMD:R_0603_1608Metric, symbol Device:R
- removed R?: 1.1k, Resistor_SMD:R_0603_1608Metric, symbol Device:R
- removed R? (x2): 4.7k, Resistor_SMD:R_0603_1608Metric, symbol Device:R
- removed R? (x2): 10k, Resistor_SMD:R_0603_1608Metric, symbol Device:R
- removed U6: TXS0104E, symbol main_board-rescue:TXS0104E-final
- removed U9: TS02CQE, Package_DIP:DIP-8_W7.62mm, symbol Analog_Switch:ADG417BN
- added C19, C22: 1µF, Capacitor_SMD:C_0603_1608Metric, symbol Device:C
- added C21: 10µF, Capacitor_SMD:C_0603_1608Metric, symbol Device:C
- added C23: 0.47µF, Capacitor_SMD:C_0603_1608Metric, symbol Device:C
- added D4: PWR, LED_SMD:LED_0805_2012Metric, symbol Device:LED_ALT
- added D6: LED, LED_SMD:LED_0805_2012Metric, symbol Device:LED_ALT
- added J5: Conn_01x02_Male, symbol Connector:Conn_01x02_Male
- added J6, J7: Conn_01x15_Male, Connector_PinHeader_2.54mm:PinHeader_1x15_P2.54mm_Vertical, symbol Connector:Conn_01x15_Male
- added R15: 1.1k, Resistor_SMD:R_0603_1608Metric, symbol Device:R
- added R18, R22, R25: 10k, Resistor_SMD:R_0603_1608Metric, symbol Device:R
- added R20, R9: 1K, Resistor_SMD:R_0603_1608Metric, symbol Device:R
- added R23, R24: 4.7k, Resistor_SMD:R_0603_1608Metric, symbol Device:R
- added R4: 10K, Resistor_SMD:R_0603_1608Metric, symbol Device:R
- added SW1: SW_DIP_x01, symbol Switch:SW_DIP_x01
- added U5: TXS0104E, symbol main_board-rescue:TXS0104E-final
- gave numbers to parts that had none: 7
- renumbered C12 to C1, C5 to C10, C15 to C11, C6 to C12, C7 to C13, C16 to C14, C8 to C15, C9 to C16, C10 to C17, C11 to C18, C17 to C2, C1 to C3, C2 to C4, C18 to C5, C3 to C6, C13 to C7, C4 to C8, C14 to C9, D5 to D3, D4 to D5, J5 to J3, J6 to J4, R11 to R1, R8 to R10, R9 to R11, R13 to R12, R14 to R13, R10 to R17, R12 to R2, R1 to R3, R4 to R6, R6 to R8, U8 to U1, U5 to U2, U1 to U3, U2 to U4, U3 to U6, U4 to U8
Connections:
- net labels removed: OUT, VPU
- wire segments 224 -> 236
- no-connect marks 42 -> 41
Other:
- moved on the sheet: C1, C10, C11, C12, C13, C14, C15, C16, C17, C18, C2, C20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

Commit message: Update Main Board
Other:
- note added: "BATTERY GAUGE"
- note added: "BATTERY HEADER"
- note added: "BATTERY MULTIPLEXER + CHARGER"
Changed lines of the file:
@@
 EESchema Schematic File Version 4
 LIBS:main_board-cache
-LIBS:sensor_board-cache
 EELAYER 26 0
 EELAYER END
@@
 Wire Wire Line
 	13450 3650 13800 3650
+Text Notes 11600 1700 0    50   ~ 0
+BATTERY MULTIPLEXER + CHARGER
+Text Notes 16050 1750 0    50   ~ 0
+BATTERY GAUGE
+Text Notes 18000 6750 0    50   ~ 0
+BATTERY HEADER
 $EndSCHEMATC

Commit message: Add inverter and change enable
Parts:
- added C?: 0.1µF, Capacitor_SMD:C_0603_1608Metric, symbol Device:C
- added U?: NC7SZ04P5X, symbol final:NC7SZ04P5X
Connections:
- wire segments 236 -> 242
Other:
- moved on the sheet: C1, C11, C14, C7, C9, D3, R1, R12, R13, R2, S2, U2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

Commit message: Linear Regulator -> Boost DC-DC
Parts:
- removed U4: MCP1702T-5002E_CB, Package_TO_SOT_SMD:SOT-23, symbol main_board-rescue:MCP1702T-5002E_CB-final
- added C24: 10µF, Capacitor_SMD:C_0603_1608Metric, symbol Device:C
- added L1: 4.7uH, symbol pspice:INDUCTOR
- added R26: 2M, Resistor_SMD:R_0603_1608Metric, symbol Device:R
- added R27: 220K, Resistor_SMD:R_0603_1608Metric, symbol Device:R
- added U4: TPS61200DRC, Package_SON:Texas_S-PVSON-N10_ThermalVias, symbol Regulator_Switching:TPS61200DRC
- C10: value 1µF -> 0.1µF
- C8: value 1µF -> 10µF
- U11: renamed from U?; symbol final:NC7SZ04P5X -> main_board-rescue:NC7SZ04P5X-final
- gave numbers to parts that had none: 1
Connections:
- wire segments 242 -> 263
Changed lines of the file:
@@
 	2700 6500 2700 6550
-$Comp
-L power:GND #PWR021
-U 1 1 5C4E24AA
-P 5250 3500
-F 0 "#PWR021" H 5250 3250 50  0001 C CNN
-F 1 "GND" H 5255 3327 50  0000 C CNN
-F 2 "" H 5250 3500 50  0001 C CNN
-F 3 "" H 5250 3500 50  0001 C CNN
-	1    5250 3500
-	1    0    0    -1
-$EndComp
 $Comp
 L power:GND #PWR037
@@
 	0    1    1    0
 $EndComp
-$Comp
-L Device:C C10
-U 1 1 5C53748B
-P 5850 3200
-F 0 "C10" H 5965 3246 50  0000 L CNN
-F 1 "1µF" H 5965 3155 50  0000 L CNN
-F 2 "Capacitor_SMD:C_0603_1608Metric" H 5888 3050 50  0001 C CNN
-F 3 "~" H 5850 3200 50  0001 C CNN
-	1    5850 3200
-	1    0    0    -1
-$EndComp
-$Comp
-L power:GND #PWR024
-U 1 1 5C5374F7
-P 5850 3350
-F 0 "#PWR024" H 5850 3100 50  0001 C CNN
-F 1 "GND" H 5855 3177 50  0000 C CNN
-F 2 "" H 5850 3350 50  0001 C CNN
-F 3 "" H 5850 3350 50  0001 C CNN
-	1    5850 3350
-	1    0    0    -1
-$EndComp
-$Comp
-L Device:C C8
-U 1 1 5C539746
-P 4650 3200
-F 0 "C8" H 4765 3246 50  0000 L CNN
-F 1 "1µF" H 4765 3155 50  0000 L CNN
-F 2 "Capacitor_SMD:C_0603_1608Metric" H 4688 3050 50  0001 C CNN
-F 3 "~" H 4650 3200 50  0001 C CNN
-	1    4650 3200
-	-1   0    0    -1
-$EndComp
-$Comp
-L power:GND #PWR016
-U 1 1 5C53B880
-P 4650 3350
-F 0 "#PWR016" H 4650 3100 50  0001 C CNN
-F 1 "GND" H 4655 3177 50  0000 C CNN
-F 2 "" H 4650 3350 50  0001 C CNN
-F 3 "" H 4650 3350 50  0001 C CNN
-	1    4650 3350
-	1    0    0    -1
-$EndComp
-Wire Wire Line
-	5750 3000 5850 3000
-Wire Wire Line
-	5850 3050 5850 3000
-Wire Wire Line
-	4750 3000 4650 3000
-Wire Wire Line
-	4650 3000 4650 3050
 Wire Wire Line
 	2650 5700 2850 5700
@@
 Wire Wire Line
 	7300 3000 7300 2600
-Wire Wire Line
-	7300 2600 5850 2600
-Wire Wire Line
-	5850 2600 5850 3000
 Connection ~ 7300 3000
 Wire Wire Line
 	7300 3000 7350 3000
-Connection ~ 5850 3000
 $Comp
 L Connector:Conn_01x15_Male J6
@@
 F 3 "" H 7950 3450 60  0001 C CNN
 	1    7950 3300
-	1    0    0    -1
-$EndComp
-$Comp
-L main_board-rescue:MCP1702T-5002E_CB-final U4
-U 1 1 5C6B8EBC
-P 5250 3100
-F 0 "U4" H 5250 3465 50  0000 C CNN
-F 1 "MCP1702T-5002E_CB" H 5250 3374 50  0000 C CNN
-F 2 "Package_TO_SOT_SMD:SOT-23" H 5250 3200 50  0001 C CNN
-F 3 "" H 5250 3200 50  0001 C CNN
-	1    5250 3100
 	1    0    0    -1
 $EndComp
@@
 Connection ~ 2450 2050
 Wire Wire Line
-	4650 3000 2200 3000
-Wire Wire Line
 	2200 3000 2200 2050
-Connection ~ 4650 3000
 Connection ~ 2200 2050
 Wire Wire Line
@@
 BATTERY HEADER
 $Comp
-L final:NC7SZ04P5X U?
+L main_board-rescue:NC7SZ04P5X-final U11
 U 1 1 5CB6DB0B
 P 7610 11260
-F 0 "U?" H 7610 11585 50  0000 C CNN
+F 0 "U11" H 7610 11585 50  0000 C CNN
 F 1 "NC7SZ04P5X" H 7610 11494 50  0000 C CNN
 F 2 "" H 7610 11260 50  0001 C CNN
@@
 $EndComp
 $Comp
-L Device:C C?
+L Device:C C25
 U 1 1 5CB7C72A
 P 7120 11410
-F 0 "C?" H 7235 11456 50  0000 L CNN
+F 0 "C25" H 7235 11456 50  0000 L CNN
 F 1 "0.1µF" H 7235 11365 50  0000 L CNN
 F 2 "Capacitor_SMD:C_0603_1608Metric" H 7158 11260 50  0001 C CNN
@@
 $EndComp
 $Comp
-L power:GND #PWR?
+L power:GND #PWR081
 U 1 1 5CB7C91F
 P 7120 11620
-F 0 "#PWR?" H 7120 11370 50  0001 C CNN
+F 0 "#PWR081" H 7120 11370 50  0001 C CNN
 F 1 "GND" V 7120 11470 50  0000 R CNN
 F 2 "" H 7120 11620 50  0001 C CNN
@@
 	7310 11260 7120 11260
 $Comp
-L power:+3V3 #PWR?
+L power:+3V3 #PWR080
 U 1 1 5CBA714F
 P 6900 11260
-F 0 "#PWR?" H 6900 11110 50  0001 C CNN
+F 0 "#PWR080" H 6900 11110 50  0001 C CNN
 F 1 "+3V3" V 6900 11410 50  0000 L CNN
 F 2 "" H 6900 11260 50  0001 C CNN
@@
 	2760 4200 2850 4200
 Connection ~ 2850 4200
+$Comp
+L Regulator_Switching:TPS61200DRC U4
+U 1 1 5CB8CDA0
+P 4750 3200
+F 0 "U4" H 4750 3667 50  0000 C CNN
+F 1 "TPS61200DRC" H 4750 3576 50  0000 C CNN
+F 2 "Package_SON:Texas_S-PVSON-N10_ThermalVias" H 4750 2750 50  0001 C CNN
+F 3 "http://www.ti.com/lit/ds/symlink/tps61200.pdf" H 4750 3200 50  0001 C CNN
+	1    4750 3200
+	1    0    0    -1
+$EndComp
+$Comp
+L Device:C C8
+U 1 1 5CB9ACC4
+P 3800 3150
+F 0 "C8" H 3915 3196 50  0000 L CNN
+F 1 "10µF" H 3915 3105 50  0000 L CNN
+F 2 "Capacitor_SMD:C_0603_1608Metric" H 3838 3000 50  0001 C CNN
+F 3 "~" H 3800 3150 50  0001 C CNN
+	1    3800 3150
+	1    0    0    -1
+$EndComp
+$Comp
+L power:GND #PWR016
+U 1 1 5CB9ACCB
+P 3800 3300
+F 0 "#PWR016" H 3800 3050 50  0001 C CNN
+F 1 "GND" H 3805 3127 50  0000 C CNN
+F 2 "" H 3800 3300 50  0001 C CNN
+F 3 "" H 3800 3300 50  0001 C CNN
+	1    3800 3300
+	1    0    0    -1
+$EndComp
+$Comp
+L power:GND #PWR021
+U 1 1 5CBC60F0
+P 4650 3800
+F 0 "#PWR021" H 4650 3550 50  0001 C CNN
+F 1 "GND" H 4655 3627 50  0000 C CNN
+F 2 "" H 4650 3800 50  0001 C CNN
+F 3 "" H 4650 3800 50  0001 C CNN
+	1    4650 3800
+	1    0    0    -1
+$EndComp
+Wire Wire Line
+	4650 3700 4650 3750
+Wire Wire Line
+	4750 3700 4750 3750
+Wire Wire Line
+	4750 3750 4650 3750
+Connection ~ 4650 3750
+Wire Wire Line
+	4650 3750 4650 3800
+Wire Wire Line
+	4850 3700 4850 3750
+Wire Wire Line
+	4850 3750 4750 3750
+Connection ~ 4750 3750
+$Comp
+L Device:C C10
+U 1 1 5CC110CE
+P 5300 3650
+F 0 "C10" H 5415 3696 50  0000 L CNN
+F 1 "0.1µF" H 5415 3605 50  0000 L CNN
+F 2 "Capacitor_SMD:C_0603_1608Metric" H 5338 3500 50  0001 C CNN
+F 3 "~" H 5300 3650 50  0001 C CNN
+	1    5300 3650
+	1    0    0    -1
+$EndComp
+$Comp
+L power:GND #PWR078
+U 1 1 5CC110D5
+P 5300 3800
+F 0 "#PWR078" H 5300 3550 50  0001 C CNN
+F 1 "GND" H 5305 3627 50  0000 C CNN
+F 2 "" H 5300 3800 50  0001 C CNN
+F 3 "" H 5300 3800 50  0001 C CNN
+	1    5300 3800
+	1    0    0    -1
+$EndComp
+$Comp
+L Device:C C24
+U 1 1 5CC308F4
+P 6100 3250
+F 0 "C24" H 6215 3296 50  0000 L CNN
+F 1 "10µF" H 6215 3205 50  0000 L CNN
+F 2 "Capacitor_SMD:C_0603_1608Metric" H 6138 3100 50  0001 C CNN
+F 3 "~" H 6100 3250 50  0001 C CNN
+	1    6100 3250
+	1    0    0    -1
+$EndComp
+$Comp
+L power:GND #PWR079
+U 1 1 5CC308FB
+P 6100 3400
+F 0 "#PWR079" H 6100 3150 50  0001 C CNN
+F 1 "GND" H 6105 3227 50  0000 C CNN
+F 2 "" H 6100 3400 50  0001 C CNN
+F 3 "" H 6100 3400 50  0001 C CNN
+	1    6100 3400
+	1    0    0    -1
+$EndComp
+Wire Wire Line
+	6100 3100 6100 2600
+Wire Wire Line
+	6100 2600 7300 2600
+Connection ~ 6100 3100
+$Comp
+L Device:R R27
+U 1 1 5CC9EFBB
+P 5750 3600
+F 0 "R27" H 5820 3646 50  0000 L CNN
+F 1 "220K" H 5820 3555 50  0000 L CNN
+F 2 "Resistor_SMD:R_0603_1608Metric" V 5680 3600 50  0001 C CNN
+F 3 "~" H 5750 3600 50  0001 C CNN
+	1    5750 3600
+	1    0    0    -1
+$EndComp
+$Comp
+L power:GND #PWR024
+U 1 1 5CC9EFC2
+P 5750 3750
+F 0 "#PWR024" H 5750 3500 50  0001 C CNN
+F 1 "GND" H 5755 3577 50  0000 C CNN
+F 2 "" H 5750 3750 50  0001 C CNN
+F 3 "" H 5750 3750 50  0001 C CNN
+	1    5750 3750
+	1    0    0    -1
+$EndComp
+$Comp
+L Device:R R26
+U 1 1 5CCDEA11
+P 5750 3250
+F 0 "R26" H 5820 3296 50  0000 L CNN
+F 1 "2M" H 5820 3205 50  0000 L CNN
+F 2 "Resistor_SMD:R_0603_1608Metric" V 5680 3250 50  0001 C CNN
+F 3 "~" H 5750 3250 50  0001 C CNN
+	1    5750 3250
+	1    0    0    -1
+$EndComp
+Wire Wire Line
+	5750 3450 5750 3400
+Connection ~ 5750 3400
+Wire Wire Line
+	4350 3300 4200 3300
+Wire Wire Line
+	4200 3300 4200 3200
+Connection ~ 4200 3000
+Wire Wire Line
+	4200 3000 4350 3000
+Wire Wire Line
+	4350 3100 4200 3100
+Connection ~ 4200 3100
+Wire Wire Line
+	4200 3100 4200 3000
+Wire Wire Line
+	4350 3200 4200 3200
+Connection ~ 4200 3200
+Wire Wire Line
+	4200 3200 4200 3100
+$Comp
+L pspice:INDUCTOR L1
+U 1 1 5CD73932
+P 4650 2600
+F 0 "L1" H 4650 2815 50  0000 C CNN
+F 1 "4.7uH" H 4650 2724 50  0000 C CNN
+F 2 "" H 4650 2600 50  0001 C CNN
+F 3 "http://products.sumida.com/products/pdf/CDRH2D18HP.pdf" H 4650 2600 50  0001 C CNN
+	1    4650 2600
+	1    0    0    -1
+$EndComp
+Wire Wire Line
+	5150 3100 5750 3100
+Connection ~ 3800 3000
+Wire Wire Line
+	3800 3000 4200 3000
+Wire Wire Line
+	4200 3000 4200 2600
+Wire Wire Line
+	4200 2600 4400 2600
+Wire Wire Line
+	5200 2600 5200 3000
+Wire Wire Line
+	5200 3000 5150 3000
+Wire Wire Line
+	4900 2600 5200 2600
+Wire Wire Line
+	2200 3000 3800 3000
+Connection ~ 5750 3100
+Wire Wire Line
+	5750 3100 6100 3100
+Wire Wire Line
+	5150 3400 5750 3400
+Wire Wire Line
+	5300 3500 5300 3200
+Wire Wire Line
+	5300 3200 5150 3200
 $EndSCHEMATC
