File: final/main_board.sch (KiCad schematic (older format))
At the start: 81 parts, among them J1 USB_microB_2040002-1, J2 Arduino_ICSP, J3 E-INK DISPLAY, J4 BT CONFIG, J5 Conn_01x02_Male, J6 Conn_01x15_Male, J7 Conn_01x15_Male, SW1 SW_DIP_x01, U1 MCP1702T-3302E/CBCT-ND, U10 BQ27441-G1, U11 NC7SZ04P5X, U2 TXS0108EPW, U3 FT232RL, U4 TPS61200DRC, U5 TXS0104E, U6 TPS2113ADRBR, U7 RN4871, U8 ATMEGA328PB-ANR, U9 BQ24075, Y1 16MHz

Commit message: Bluetooth Power LED Footprint Assigned
Parts:
- D3: footprint (none) -> LED_SMD:LED_0805_2012Metric
- J3: footprint Connector_JST:JST_EH_B08B-EH-A_1x08_P2.50mm_Vertical -> (none)
Changed lines of the file:
@@
 F 0 "J3" H 19762 11633 50  0000 R CNN
 F 1 "E-INK DISPLAY" H 19762 11542 50  0000 R CNN
-F 2 "Connector_JST:JST_EH_B08B-EH-A_1x08_P2.50mm_Vertical" H 19790 11660 50  0001 C CNN
+F 2 "" H 19790 11660 50  0001 C CNN
 F 3 "~" H 19790 11660 50  0001 C CNN
 	1    19790 11660
@@
 F 0 "D3" H 11971 12026 50  0000 C CNN
 F 1 "BTPWR" H 11971 11935 50  0000 C CNN
-F 2 "" H 11980 11810 50  0001 C CNN
+F 2 "LED_SMD:LED_0805_2012Metric" H 11980 11810 50  0001 C CNN
 F 3 "~" H 11980 11810 50  0001 C CNN
 	1    11980 11810

Commit message: Add assignment for small logic converter
Parts:
- D3: footprint LED_SMD:LED_0805_2012Metric -> (none)
- J3: footprint (none) -> Connector_JST:JST_EH_B08B-EH-A_1x08_P2.50mm_Vertical
- U5: footprint (none) -> mp3b:txs0104e
Changed lines of the file:
@@
 F 0 "J3" H 19762 11633 50  0000 R CNN
 F 1 "E-INK DISPLAY" H 19762 11542 50  0000 R CNN
-F 2 "" H 19790 11660 50  0001 C CNN
+F 2 "Connector_JST:JST_EH_B08B-EH-A_1x08_P2.50mm_Vertical" H 19790 11660 50  0001 C CNN
 F 3 "~" H 19790 11660 50  0001 C CNN
 	1    19790 11660
@@
 F 0 "D3" H 11971 12026 50  0000 C CNN
 F 1 "BTPWR" H 11971 11935 50  0000 C CNN
-F 2 "LED_SMD:LED_0805_2012Metric" H 11980 11810 50  0001 C CNN
+F 2 "" H 11980 11810 50  0001 C CNN
 F 3 "~" H 11980 11810 50  0001 C CNN
 	1    11980 11810
@@
 F 0 "U5" H 8985 11004 50  0000 C CNN
 F 1 "TXS0104E" H 8985 10913 50  0000 C CNN
-F 2 "" H 9210 11640 50  0001 C CNN
+F 2 "mp3b:txs0104e" H 9210 11640 50  0001 C CNN
 F 3 "" H 9210 11640 50  0001 C CNN
 	1    9010 11640

Commit message: Final Footprints
Parts:
- D3: footprint (none) -> LED_SMD:LED_0805_2012Metric
Changed lines of the file:
@@
 F 0 "D3" H 11971 12026 50  0000 C CNN
 F 1 "BTPWR" H 11971 11935 50  0000 C CNN
-F 2 "" H 11980 11810 50  0001 C CNN
+F 2 "LED_SMD:LED_0805_2012Metric" H 11980 11810 50  0001 C CNN
 F 3 "~" H 11980 11810 50  0001 C CNN
 	1    11980 11810

Commit message: Change jst footprint assignment
Parts:
- J3: footprint Connector_JST:JST_EH_B08B-EH-A_1x08_P2.50mm_Vertical -> Connector_JST:JST_PH_B8B-PH-SM4-TB_1x08-1MP_P2.00mm_Vertical
Changed lines of the file:
@@
 F 0 "J3" H 19762 11633 50  0000 R CNN
 F 1 "E-INK DISPLAY" H 19762 11542 50  0000 R CNN
-F 2 "Connector_JST:JST_EH_B08B-EH-A_1x08_P2.50mm_Vertical" H 19790 11660 50  0001 C CNN
+F 2 "Connector_JST:JST_PH_B8B-PH-SM4-TB_1x08-1MP_P2.00mm_Vertical" H 19790 11660 50  0001 C CNN
 F 3 "~" H 19790 11660 50  0001 C CNN
 	1    19790 11660

Commit message: Add ground pad to QFNs
Parts:
- U3: symbol main_board-rescue:FT232RL-final -> final:FT232RL
- U8: symbol main_board-rescue:ATMEGA328PB-ANR-final -> final:ATMEGA328PB-ANR
Connections:
- wire segments 263 -> 266
Changed lines of the file:
@@
 $EndComp
 $Comp
-L main_board-rescue:ATMEGA328PB-ANR-final U8
+L final:ATMEGA328PB-ANR U8
 U 1 1 5C6C352E
 P 10250 7200
@@
 	9100 8900 9100 8950
 $Comp
-L main_board-rescue:FT232RL-final U3
+L final:FT232RL U3
 U 1 1 5C6CF653
 P 4950 6600
@@
 Wire Wire Line
 	5300 3200 5150 3200
+Wire Wire Line
+	9250 8300 9100 8300
+Wire Wire Line
+	9100 8300 9100 8500
+Connection ~ 9100 8500
+$Comp
+L power:GND #PWR?
+U 1 1 5CC0504C
+P 5250 8200
+F 0 "#PWR?" H 5250 7950 50  0001 C CNN
+F 1 "GND" H 5255 8027 50  0000 C CNN
+F 2 "" H 5250 8200 50  0001 C CNN
+F 3 "" H 5250 8200 50  0001 C CNN
+	1    5250 8200
+	1    0    0    -1
+$EndComp
+Wire Wire Line
+	5250 8200 5250 8100
 $EndSCHEMATC

Commit message: Update 1
Parts:
- removed J6, J7: Conn_01x15_Male, Connector_PinHeader_2.54mm:PinHeader_1x15_P2.54mm_Vertical, symbol Connector:Conn_01x15_Male
- U3: symbol final:FT232RL -> main_board-rescue:FT232RL-final
- U8: symbol final:ATMEGA328PB-ANR -> main_board-rescue:ATMEGA328PB-ANR-final
Connections:
- wire segments 266 -> 259
- no-connect marks 41 -> 52
Changed lines of the file:
@@
 Wire Wire Line
 	7300 3000 7350 3000
-$Comp
-L Connector:Conn_01x15_Male J6
-U 1 1 5CB10A94
-P 19800 7850
-F 0 "J6" H 19773 7873 50  0000 R CNN
-F 1 "Conn_01x15_Male" H 19773 7782 50  0000 R CNN
-F 2 "Connector_PinHeader_2.54mm:PinHeader_1x15_P2.54mm_Vertical" H 19800 7850 50  0001 C CNN
-F 3 "~" H 19800 7850 50  0001 C CNN
-	1    19800 7850
-	-1   0    0    -1
-$EndComp
-$Comp
-L Connector:Conn_01x15_Male J7
-U 1 1 5CB10A95
-P 19800 9650
-F 0 "J7" H 19773 9673 50  0000 R CNN
-F 1 "Conn_01x15_Male" H 19773 9582 50  0000 R CNN
-F 2 "Connector_PinHeader_2.54mm:PinHeader_1x15_P2.54mm_Vertical" H 19800 9650 50  0001 C CNN
-F 3 "~" H 19800 9650 50  0001 C CNN
-	1    19800 9650
-	-1   0    0    -1
-$EndComp
-Text Label 19600 7150 2    50   ~ 0
-VIN
-$Comp
-L power:GND #PWR072
-U 1 1 5C586795
-P 19400 7250
-F 0 "#PWR072" H 19400 7000 50  0001 C CNN
-F 1 "GND" V 19400 7100 50  0000 R CNN
-F 2 "" H 19400 7250 50  0001 C CNN
-F 3 "" H 19400 7250 50  0001 C CNN
-	1    19400 7250
-	0    1    1    0
-$EndComp
-Text Label 19600 7350 2    50   ~ 0
-RESET
-$Comp
-L power:+5V #PWR073
-U 1 1 5C59157E
-P 19400 7450
-F 0 "#PWR073" H 19400 7300 50  0001 C CNN
-F 1 "+5V" V 19400 7600 50  0000 L CNN
-F 2 "" H 19400 7450 50  0001 C CNN
-F 3 "" H 19400 7450 50  0001 C CNN
-	1    19400 7450
-	0    -1   -1   0
-$EndComp
-Text Label 19600 7550 2    50   ~ 0
-A7
-Text Label 19600 7650 2    50   ~ 0
-A6
-Text Label 19600 7750 2    50   ~ 0
-A5
-Text Label 19600 7850 2    50   ~ 0
-A4
-Text Label 19600 7950 2    50   ~ 0
-A3
-Text Label 19600 8050 2    50   ~ 0
-A2
-Text Label 19600 8150 2    50   ~ 0
-A1
-Text Label 19600 8250 2    50   ~ 0
-A0
-Wire Wire Line
-	19400 7450 19600 7450
-Wire Wire Line
-	19400 7250 19600 7250
 Text Label 9150 6900 2    50   ~ 0
-AREF
-Text Label 19600 8350 2    50   ~ 0
 AREF
 $Comp
@@
 	0    -1   1    0
 $EndComp
-Wire Wire Line
-	19400 8450 19600 8450
-Text Label 19600 8950 2    50   ~ 0
-D1
-Text Label 19600 9050 2    50   ~ 0
-D0
-Text Label 19600 9150 2    50   ~ 0
-RESET
-$Comp
-L power:GND #PWR075
-U 1 1 5CB10A98
-P 19400 9250
-F 0 "#PWR075" H 19400 9000 50  0001 C CNN
-F 1 "GND" V 19400 9100 50  0000 R CNN
-F 2 "" H 19400 9250 50  0001 C CNN
-F 3 "" H 19400 9250 50  0001 C CNN
-	1    19400 9250
-	0    1    1    0
-$EndComp
-Wire Wire Line
-	19400 9250 19600 9250
-Text Label 19600 9350 2    50   ~ 0
-D2
-Text Label 19600 9450 2    50   ~ 0
-D3
-Text Label 19600 9550 2    50   ~ 0
-D4
-Text Label 19600 9650 2    50   ~ 0
-D5
-Text Label 19600 9750 2    50   ~ 0
-D6
-Text Label 19600 10350 2    50   ~ 0
-D12
 Text Label 19470 10730 2    50   ~ 0
 D12
@@
 $EndComp
 $Comp
-L final:ATMEGA328PB-ANR U8
+L main_board-rescue:ATMEGA328PB-ANR-final U8
 U 1 1 5C6C352E
 P 10250 7200
@@
 	9100 8900 9100 8950
 $Comp
-L final:FT232RL U3
+L main_board-rescue:FT232RL-final U3
 U 1 1 5C6CF653
 P 4950 6600
@@
 NoConn ~ 4050 11500
 NoConn ~ 4050 11600
+Text Label 4850 11300 0    50   ~ 0
+D11
+Text Label 4850 11400 0    50   ~ 0
+D13
+Text Label 4850 11200 0    50   ~ 0
+D10
+Text Label 4850 11100 0    50   ~ 0
+D9
+Text Label 4850 11000 0    50   ~ 0
+D8
 Text Label 4850 10900 0    50   ~ 0
-D11
-Text Label 4850 11000 0    50   ~ 0
-D13
-Text Label 4850 11100 0    50   ~ 0
-D10
-Text Label 4850 11200 0    50   ~ 0
-D9
-Text Label 4850 11300 0    50   ~ 0
-D8
-Text Label 4850 11400 0    50   ~ 0
 D7
 NoConn ~ 4850 11500
@@
 CTS
 NoConn ~ 10140 11910
-Text Label 19600 8550 2    50   ~ 0
-D13
-Text Label 19600 10250 2    50   ~ 0
-D11
-Text Label 19600 10150 2    50   ~ 0
-D10
-Text Label 19600 10050 2    50   ~ 0
-D9
-Text Label 19600 9950 2    50   ~ 0
-D8
-Text Label 19600 9850 2    50   ~ 0
-D7
 Text Notes 18970 11240 0    50   ~ 0
 8-Pin JST rectangular \nconnector for E-Ink display
@@
 Bluetooth module
 $Comp
-L power:+3V3 #PWR074
-U 1 1 5CB62328
-P 19400 8450
-F 0 "#PWR074" H 19400 8300 50  0001 C CNN
-F 1 "+3V3" V 19400 8600 50  0000 L CNN
-F 2 "" H 19400 8450 50  0001 C CNN
-F 3 "" H 19400 8450 50  0001 C CNN
-	1    19400 8450
-	0    -1   1    0
-$EndComp
-$Comp
 L power:GND #PWR05
 U 1 1 5CAC31DC
@@
 Wire Wire Line
 	5300 3200 5150 3200
-Wire Wire Line
-	9250 8300 9100 8300
-Wire Wire Line
-	9100 8300 9100 8500
-Connection ~ 9100 8500
-$Comp
-L power:GND #PWR?
-U 1 1 5CC0504C
-P 5250 8200
-F 0 "#PWR?" H 5250 7950 50  0001 C CNN
-F 1 "GND" H 5255 8027 50  0000 C CNN
-F 2 "" H 5250 8200 50  0001 C CNN
-F 3 "" H 5250 8200 50  0001 C CNN
-	1    5250 8200
-	1    0    0    -1
-$EndComp
-Wire Wire Line
-	5250 8200 5250 8100
+NoConn ~ 11350 9100
+NoConn ~ 11350 8900
+NoConn ~ 11350 8700
+NoConn ~ 11350 8500
+NoConn ~ 11350 8300
+NoConn ~ 11350 6700
+NoConn ~ 11350 6500
+NoConn ~ 11350 6300
+NoConn ~ 11350 6100
+NoConn ~ 11350 5900
+NoConn ~ 11350 5700
 $EndSCHEMATC

Commit message: Final_Push
Parts:
- U3: symbol main_board-rescue:FT232RL-final -> sensor_board-rescue:FT232RL-final
- U8: symbol main_board-rescue:ATMEGA328PB-ANR-final -> sensor_board-rescue:ATMEGA328PB-ANR-final
Changed lines of the file:
@@
 $EndComp
 $Comp
-L main_board-rescue:ATMEGA328PB-ANR-final U8
+L sensor_board-rescue:ATMEGA328PB-ANR-final U8
 U 1 1 5C6C352E
 P 10250 7200
@@
 	9100 8900 9100 8950
 $Comp
-L main_board-rescue:FT232RL-final U3
+L sensor_board-rescue:FT232RL-final U3
 U 1 1 5C6CF653
 P 4950 6600
@@
 NoConn ~ 11350 5900
 NoConn ~ 11350 5700
+$Comp
+L power:GND #PWR?
+U 1 1 5CC0974F
+P 5250 8200
+F 0 "#PWR?" H 5250 7950 50  0001 C CNN
+F 1 "GND" H 5255 8027 50  0000 C CNN
+F 2 "" H 5250 8200 50  0001 C CNN
+F 3 "" H 5250 8200 50  0001 C CNN
+	1    5250 8200
+	1    0    0    -1
+$EndComp
+Wire Wire Line
+	5250 8100 5250 8200
+Wire Wire Line
+	9250 8300 9100 8300
+Wire Wire Line
+	9100 8300 9100 8500
+Connection ~ 9100 8500
 $EndSCHEMATC

Commit message: changes to senor layout
Parts:
- U3: symbol sensor_board-rescue:FT232RL-final -> main_board-rescue:FT232RL-final-sensor_board-rescue
- U8: symbol sensor_board-rescue:ATMEGA328PB-ANR-final -> main_board-rescue:ATMEGA328PB-ANR-final-sensor_board-rescue
Connections:
- net GND: now also U3.33 (GND), U8.33 (GND)
Changed lines of the file:
@@
 EESchema Schematic File Version 4
 LIBS:main_board-cache
-EELAYER 26 0
+EELAYER 29 0
 EELAYER END
 $Descr C 22000 17000
@@
 $EndComp
 $Comp
-L sensor_board-rescue:ATMEGA328PB-ANR-final U8
+L main_board-rescue:ATMEGA328PB-ANR-final-sensor_board-rescue U8
 U 1 1 5C6C352E
 P 10250 7200
@@
 	9100 8900 9100 8950
 $Comp
-L sensor_board-rescue:FT232RL-final U3
+L main_board-rescue:FT232RL-final-sensor_board-rescue U3
 U 1 1 5C6CF653
 P 4950 6600
