File: final/main_board.kicad_pcb (KiCad board)
At the start: 2 copper layers, 81 parts, among them J1 USB_microB_2040002-1, J2 Arduino_ICSP, J3 E-INK DISPLAY, J4 BT CONFIG, J5 Conn_01x02_Male, J6 Conn_01x15_Male, J7 Conn_01x15_Male, SW1 SW_DIP_x01, U1 MCP1702T-3302E/CBCT-ND, U10 BQ27441-G1, U11 NC7SZ04P5X, U2 TXS0108EPW, U3 FT232RL, U4 TPS61200DRC, U5 TXS0104E, U6 TSP2113ADRBR, U7 RN4871, U8 ATMEGA328PB-ANR, U9 BQ24075, Y1 16MHz

Commit message: Layout
Parts:
- moved J4 177.7 mm to (222.6, 112.5)
- moved R10 132.5 mm to (176.4, 154.7)
- moved J6 119.6 mm to (126.7, 109.1)
- moved J3 115.7 mm to (60.3, 146.6)
- moved R13 111.1 mm to (173.9, 114.8)
- moved S1 110.3 mm to (176.3, 151.5)
- moved J7 100.7 mm to (83.0, 112.1)
- moved J2 94.7 mm to (57.3, 135.7)
- moved D3 92.9 mm to (108.0, 145.8), turned to 90 degrees
- moved U7 91.9 mm to (114.6, 149.6), turned to 180 degrees
- moved C2 90.9 mm to (100.2, 123.6), turned to 90 degrees
- moved SW1 89.4 mm to (105.3, 174.9), turned to 90 degrees
- moved C1 86.1 mm to (79.4, 141.7), turned to 180 degrees
- moved R2 84.6 mm to (103.6, 135.4), turned to 270 degrees
- moved C9 84.5 mm to (104.1, 142.1), turned to 180 degrees
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Routing:
- net /D9: track 0.00 -> 18.8 mm
- net /D12: track 0.00 -> 17.5 mm
- net /D8: track 0.00 -> 16.3 mm
- net /D11: track 0.00 -> 15.0 mm
- net /BATTERY: track 0.00 -> 14.5 mm
- net /D10: track 0.00 -> 12.7 mm
- net GND: track 0.00 -> 12.7 mm
- net /D5: track 0.00 -> 6.79 mm
- net /D7: track 0.00 -> 6.61 mm
- net /D6: track 0.00 -> 6.25 mm
- net +5V: track 0.00 -> 3.84 mm
- net /A4: track 0.00 -> 2.57 mm
- net Net-(R25-Pad1): track 0.00 -> 2.11 mm
- net /V_BATT: track 0.00 -> 2.03 mm
- net Net-(C23-Pad1): track 0.00 -> 1.86 mm
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Other:
- rule trace_min: 0.2 -> 0.1524

Commit message: Updated Layout
Parts:
- moved C9 27.5 mm to (95.1, 116.2), turned to 0 degrees
- moved C25 21.5 mm to (95.3, 113.1)
- moved U11 21.4 mm to (93.4, 113.2)
- moved U5 20.4 mm to (96.3, 121.5), turned to 270 degrees
- moved R2 19.9 mm to (98.3, 116.2), turned to 180 degrees
- moved C11 18.1 mm to (98.4, 127.0), turned to 0 degrees
- moved R24 15.9 mm to (128.1, 110.2)
- moved C23 15.9 mm to (130.2, 106.7)
- moved J5 15.9 mm to (127.9, 97.4)
- moved R21 15.9 mm to (125.0, 104.8)
- moved R22 15.9 mm to (123.4, 107.1)
- moved R23 15.9 mm to (130.5, 109.2)
- moved R25 15.9 mm to (124.9, 110.2)
- moved U10 15.9 mm to (127.0, 107.5)
- moved C22 15.9 mm to (128.1, 104.8)
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Routing:
- net GND: track 12.7 -> 32.6 mm
- net +5V: track 3.84 -> 23.0 mm
- net Net-(C2-Pad1): track 0.00 -> 13.8 mm
- net /RESET: track 0.00 -> 12.3 mm
- net /D0: track 0.00 -> 11.8 mm
- net Net-(C24-Pad1): track 0.00 -> 11.0 mm
- net /D3: track 0.00 -> 10.9 mm
- net /UART_EN: track 0.00 -> 9.66 mm
- net /D4: track 0.00 -> 9.40 mm
- net Net-(L1-Pad2): track 0.00 -> 6.96 mm
- net Net-(R26-Pad2): track 0.00 -> 6.68 mm
- net Net-(R4-Pad2): track 0.00 -> 4.81 mm
- net +3V3: track 0.00 -> 4.47 mm
- net Net-(R5-Pad1): track 0.00 -> 2.61 mm
- net Net-(U8-Pad8): track 0.00 -> 2.55 mm
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
Commit message: Update 1
Parts:
- removed J6, J7: Conn_01x15_Male, Connector_PinHeader_2.54mm:PinHeader_1x15_P2.54mm_Vertical
- U6: value TSP2113ADRBR -> TPS2113ADRBR
- moved J4 108.4 mm to (115.4, 128.5)
- moved R10 101.0 mm to (78.4, 130.2)
- moved S1 101.0 mm to (78.4, 127.0)
- moved R13 72.8 mm to (109.0, 147.6)
- moved S2 66.5 mm to (109.9, 145.0)
- moved SW1 65.1 mm to (115.7, 110.7), turned to 0 degrees
- moved R23 31.8 mm to (102.2, 123.7), turned to 0 degrees
- moved C23 30.5 mm to (104.7, 123.5), turned to 180 degrees
- moved R24 29.1 mm to (101.2, 121.4), turned to 270 degrees
- moved J2 29.0 mm to (86.4, 136.6)
- moved J5 27.6 mm to (114.0, 121.2), turned to 270 degrees
- moved C22 27.1 mm to (106.6, 121.4), turned to 270 degrees
- moved U10 26.4 mm to (103.9, 120.2), turned to 90 degrees
- moved J3 26.3 mm to (86.6, 145.3)
- moved R25 25.0 mm to (101.2, 118.2), turned to 270 degrees
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Connections:
- U2 pad 14: /D7 -> /D13
- U2 pad 15: /D8 -> /D11
- U2 pad 16: /D9 -> /D10
- U2 pad 17: /D10 -> /D9
- U2 pad 18: /D13 -> /D8
- U2 pad 20: /D11 -> /D7
Routing:
- net +3V3: track 4.47 -> 24.1 mm
- net /D13: track 0.00 -> 19.3 mm
- net /D9: track 18.8 -> 1.96 mm
- net /DIN: track 0.00 -> 15.7 mm
- net /D8: track 16.3 -> 1.92 mm
- net /BUSY: track 0.00 -> 14.2 mm
- net Net-(J1-Pad3): track 0.00 -> 13.7 mm, vias 0 -> 2
- net /A4: track 2.57 -> 15.9 mm, vias 0 -> 2
- net /UART_EN: track 9.66 -> 22.8 mm, vias 0 -> 2
- net /~RST: track 0.00 -> 13.1 mm, vias 0 -> 1
- net /A5: track 1.66 -> 14.7 mm
- net Net-(J1-Pad2): track 0.00 -> 12.8 mm, vias 0 -> 2
- net /RST: track 0.00 -> 12.3 mm
- net /CTS: track 0.00 -> 11.7 mm, vias 0 -> 1
- net /D3: track 10.9 -> 0.00 mm
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
Commit message: Update 2
Parts:
- moved S1 27.9 mm to (102.8, 113.6), turned to 180 degrees
- moved R10 25.0 mm to (99.1, 116.1)
- moved R11 6.44 mm to (100.7, 107.0), turned to 90 degrees
- moved D4 3.86 mm to (98.5, 109.8)
- moved C8 3.86 mm to (101.9, 111.1)
- moved C24 3.61 mm to (101.9, 109.4), turned to 180 degrees
- moved C5 3.58 mm to (109.3, 106.1)
- moved U1 3.52 mm to (109.5, 108.8)
- moved C2 3.48 mm to (109.3, 111.5)
- moved R23 3.14 mm to (100.4, 121.1)
- moved R27 2.87 mm to (104.8, 106.1)
- moved C10 2.87 mm to (104.8, 107.7)
- moved R26 2.87 mm to (102.4, 107.0)
- moved U4 2.87 mm to (105.6, 110.2)
- moved R24 2.06 mm to (100.4, 119.5), turned to 180 degrees
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Routing:
- net GND: track 38.0 -> 145.9 mm, vias 0 -> 15
- net +3V3: track 24.1 -> 125.2 mm, vias 0 -> 5
- net +5V: track 33.6 -> 90.9 mm, vias 0 -> 9
- net /RESET: track 4.86 -> 40.7 mm, vias 1 -> 3
- net /RX: track 5.48 -> 31.2 mm, vias 0 -> 2
- net /TX: track 5.06 -> 30.4 mm, vias 1 -> 3
- net /V_BATT: track 4.82 -> 25.7 mm, vias 0 -> 2
- net /VIN: track 4.44 -> 24.3 mm, vias 0 -> 2
- net /UART_EN: track 22.8 -> 40.2 mm, vias 2 -> 4
- net /~RST: track 13.1 -> 20.1 mm, vias 1 -> 2
- net Net-(D3-Pad1): track 0.00 -> 5.61 mm
- net Net-(R18-Pad1): track 0.00 -> 4.28 mm
- net Net-(L1-Pad2): track 6.96 -> 10.6 mm
- net Net-(J1-Pad3): track 13.7 -> 16.3 mm
- net /AREF: track 0.00 -> 2.09 mm
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- added copper zone on F.Cu, net +3V3
- added copper zone on B.Cu, net GND

Commit message: Final_Push
Parts:
- moved J1 2.43 mm to (88.4, 106.7), turned to 180 degrees
- moved C18 0.13 mm to (86.2, 126.8)
Connections:
- U3 pad 33: (no net) -> GND
- U8 pad 33: (no net) -> GND
Routing:
- net GND: track 145.9 -> 167.2 mm, vias 15 -> 16
- net /D0: track 9.74 -> 28.9 mm, vias 1 -> 2
- net +3V3: track 125.2 -> 113.5 mm
- net /UART_EN: track 40.2 -> 33.9 mm
- net /RESET: track 40.7 -> 38.9 mm
- net +5V: track 90.9 -> 92.3 mm
- net Net-(J1-Pad2): track 14.5 -> 15.9 mm
- net Net-(U8-Pad7): track 3.98 -> 5.20 mm
- net /D1: track 9.25 -> 10.0 mm
- net Net-(J1-Pad3): track 16.3 -> 15.5 mm
Other:
- board outline added: 34.5 x 43.7 mm

Commit message: Update 3
Routing:
- net +3V3: track 113.5 -> 78.5 mm
- net GND: track 167.2 -> 165.8 mm
- net /VIN: track 24.3 -> 25.0 mm
- net /V_BATT: track 25.7 -> 25.0 mm
- net /D1: track 10.0 -> 9.50 mm
- net +5V: track 92.3 -> 92.9 mm
